Commit message: Flip X carriage to match Y stage and guard slide travel specs
The Onshape export mounted the X-stage carriage as a 180 deg mirror of
the Y-stage carriage (encoder/readhead toward base -x, home-limit
switch/flag toward base +x). Rotate the whole X carriage subtree 180 deg
about the vertical axis through the carriage centre so it is posed
exactly like the Y carriage (encoder toward base +x, switch/flag toward
base -x); carriage stays upright and travel still follows world +X.

Anchoring the flip on the carriage centre (not the mount) keeps the X
carriage at the same along-slide position as Y (q_mid +20.733 mm) and
puts the X home-limit trip at +11.9 mm like Y, so home_offset.py now
measures the X stage with the flipped pose map.

Add generator verification guards so the declared travel cannot silently
drift from the Parker 401200XR spec: both slides must have exactly
200 mm stroke and stay centred on the physical mid-stroke, recomputed
from mesh geometry.

Regenerate parkerstage.urdf and the doc SVGs; update README home and
caveat text.

Generated with Codebuff 🤖
Co-Authored-By: Codebuff <noreply@codebuff.com>

File: urdf/parkerstage.urdf (robot description, URDF)
Before this commit: robot parkerstage, 17 links, 16 joints
Joints:
- joint x_slide: axis -1 0 0 -> 1 0 0; origin xyz=0 -0.03345 -0.02135 rpy=1.5708 0 -1.570796 -> xyz=0 -0.03405 -0.02135 rpy=1.5708 0 1.570796

Commit message: Add 401XR150 Z axis to make parkerstage an XYZ compound stage
Mount the Parker 401XR 150 vertically on the X carriage (motor up, base
-z end down) and drive it with a new z_slide prismatic along world +Z
(150 mm stroke, limits [-0.0540, +0.0960] centered on the physical
mid-stroke +21.030 mm, home trip +11.912 mm).  The generator now parses
the second Onshape export (urdf/zslide.urdf.onshape), namespaces its
meshes, mounts the Z base on the X carriage centre, and adds 10 Z
collision boxes; verify() gains the world-Z axis, 150 mm stroke,
mid-stroke and home guards plus a 3-axis 125-config collision sweep
(zero overlaps over 900 box pairs).  home_offset.py measures the Z
stage; the kinematic-tree and collision-geometry SVGs render the Z
branch (including a fix for the collision figure's metre-scale panel
padding that made every box sub-pixel), the 3D viewer drives all three
slides, and the README/package.xml describe the XYZ model.

🤖 Generated with Codebuff
Co-Authored-By: Codebuff <noreply@codebuff.com>

File: urdf/parkerstage.urdf (robot description, URDF)
Before this commit: robot parkerstage, 17 links, 16 joints
Links:
- added link z_10851610__10851610, mass 0.0716742; visual mesh filename=package://parkerstage/meshes/z__10851610__10851610.stl scale=1 1 1
- added link z_401xr_150_base__401xr_150_base, mass 0.3673404; collision box size=0.01477 0.03329 0.267; collision box size=0.01513 0.03329 0.267
- added link z_401xr_150_seal_seal__401xr_150_seal_seal, mass 0.0121824; visual mesh filename=package://parkerstage/meshes/z__401XR_150_Seal_seal__401XR_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 scale=1 1 1
- added link z_401xr___150___d9___drive_screw__401xr___150___d9___drive_screw, mass 0.0258876; visual mesh filename=package://parkerstage/meshes/z__401XR___150___D9___Drive_Sc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 scale=1 1 1
- added link z_401xr___carriage__401xr___carriage, mass 0.0634284; collision box size=0.008 0.009 0.045; visual mesh filename=package://parkerstage/meshes/z__401XR___Carriage__401XR___C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 scale=1 1 1
- added link z_401xr___carriage_end_caps__401xr___carriage_end_caps, mass 0.0323865; collision box size=0.008 0.007 0.0236; collision box size=0.008 0.007 0.0237
- added link z_401xr___carriage_end_caps__401xr___carriage_end_caps_1__1_, mass 1e-09
- added link z_401xr___encoder__401xr___encoder, mass 0.0346221; collision box size=0.014 0.031 0.0445; visual mesh filename=package://parkerstage/meshes/z__401XR___Encoder__401XR___En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 scale=1 1 1
- added link z_401xr___encoder_base_2__401xr___encoder_base_2, mass 0.0031455; visual mesh filename=package://parkerstage/meshes/z__401XR___Encoder_Base_2__401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 scale=1 1 1
- added link z_401xr___encoder_base_2__401xr___encoder_base_2_1, mass 0.0031617; collision box size=0.0065 0.0075 0.0135; visual mesh filename=package://parkerstage/meshes/z__401XR___Encoder_Base_2__401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 scale=1 1 1
- added link z_401xr___h2__l1___homelimit_switch__401xr___h2__l1___homelimit_switch, mass 0.0047223; collision box size=0.0055 0.0095 0.0345; visual mesh filename=package://parkerstage/meshes/z__401XR___H2__L1___Homelimit_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 scale=1 1 1
- added link z_401xr___h2__l2___homelimit_switch__401xr___h2__l2___homelimit_switch_1, mass 0.0111915; visual mesh filename=package://parkerstage/meshes/z__401XR___H2__L2___Homelimit_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 scale=1 1 1
- added link z_401xr___h2__l2___homelimit_switch__401xr___h2__l2___homelimit_switch__1_, mass 1e-09
- added link z_401xr___switch_flag__401xr___switch_flag, mass 0.0008991; collision box size=0.0075 0.009 0.015; visual mesh filename=package://parkerstage/meshes/z__401XR___Switch_Flag__401XR_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 scale=1 1 1
- added link z_401xr_back_ballscrew_holder__401xr_back_ballscrew_holder, mass 0.0151011; visual mesh filename=package://parkerstage/meshes/z__401XR_Back_Ballscrew_Holder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 scale=1 1 1
- added link z_401xr_coupling_housing__401xr_coupling_housing, mass 0.1522071; visual mesh filename=package://parkerstage/meshes/z__401XR_Coupling_Housing__401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 scale=1 1 1
- added link z_401xr_front_ballscrew_holder__401xr_front_ballscrew_holder, mass 0.0344223; visual mesh filename=package://parkerstage/meshes/z__401XR_Front_Ballscrew_Holde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 scale=1 1 1
- added link z_c3_401xr__c3_401xr, mass 0.0190296; visual mesh filename=package://parkerstage/meshes/z_C3_401XR__C3_401XR.stl scale=1 1 1
- added link z_m2___sm_16__m2___sm_16, mass 0.0035235; visual mesh filename=package://parkerstage/meshes/z_M2___SM_16__M2___SM_16.stl scale=1 1 1
Joints:
- added joint z_group_1_fastened_joint: type fixed, parent z_c3_401xr__c3_401xr, child z_401xr_front_ballscrew_holder__401xr_front_ballscrew_holder, origin xyz=0 0 0 rpy=0 -0 0
- added joint z_group_1_fastened_joint_1: type fixed, parent z_401xr___150___d9___drive_screw__401xr___150___d9___drive_screw, child z_10851610__10851610, origin xyz=0 0 0 rpy=0 -0 0
- added joint z_group_1_fastened_joint_10: type fixed, parent z_c3_401xr__c3_401xr, child z_m2___sm_16__m2___sm_16, origin xyz=0 0 0 rpy=0 -0 0
- added joint z_group_1_fastened_joint_2: type fixed, parent z_401xr___h2__l2___homelimit_switch__401xr___h2__l2___homelimit_switch_1, child z_401xr___h2__l2___homelimit_switch__401xr___h2__l2___homelimit_switch__1_, origin xyz=0 0 0 rpy=0 -0 0
- added joint z_group_1_fastened_joint_3: type fixed, parent z_401xr___encoder_base_2__401xr___encoder_base_2, child z_401xr___150___d9___drive_screw__401xr___150___d9___drive_screw, origin xyz=0 0 0 rpy=0 -0 0
- added joint z_group_1_fastened_joint_4: type fixed, parent z_401xr_back_ballscrew_holder__401xr_back_ballscrew_holder, child z_401xr_150_seal_seal__401xr_150_seal_seal, origin xyz=0 0 0 rpy=0 -0 0
- added joint z_group_1_fastened_joint_5: type fixed, parent z_401xr_coupling_housing__401xr_coupling_housing, child z_401xr_back_ballscrew_holder__401xr_back_ballscrew_holder, origin xyz=0 0 0 rpy=0 -0 0
- added joint z_group_1_fastened_joint_6: type fixed, parent z_401xr_front_ballscrew_holder__401xr_front_ballscrew_holder, child z_401xr_coupling_housing__401xr_coupling_housing, origin xyz=0 0 0 rpy=0 -0 0
- added joint z_group_1_fastened_joint_7: type fixed, parent z_401xr_150_base__401xr_150_base, child z_401xr___h2__l2___homelimit_switch__401xr___h2__l2___homelimit_switch_1, origin xyz=0 0 0 rpy=0 -0 0
- added joint z_group_1_fastened_joint_8: type fixed, parent z_401xr___h2__l2___homelimit_switch__401xr___h2__l2___homelimit_switch__1_, child z_401xr___encoder_base_2__401xr___encoder_base_2, origin xyz=0 0 0 rpy=0 -0 0
- added joint z_group_1_fastened_joint_9: type fixed, parent z_401xr_150_seal_seal__401xr_150_seal_seal, child z_401xr_150_base__401xr_150_base, origin xyz=0 0 0 rpy=0 -0 0
- added joint z_group_2_fastened_joint: type fixed, parent z_401xr___carriage_end_caps__401xr___carriage_end_caps_1__1_, child z_401xr___carriage_end_caps__401xr___carriage_end_caps, origin xyz=0 0 0 rpy=0 -0 0
- added joint z_group_2_fastened_joint_1: type fixed, parent z_401xr___carriage__401xr___carriage, child z_401xr___carriage_end_caps__401xr___carriage_end_caps_1__1_, origin xyz=-0.0213302 -0.02125 -0.020468 rpy=0 -0 0
- added joint z_group_2_fastened_joint_2: type fixed, parent z_401xr___h2__l1___homelimit_switch__401xr___h2__l1___homelimit_switch, child z_401xr___switch_flag__401xr___switch_flag, origin xyz=0 0 0 rpy=0 -0 0
- added joint z_group_2_fastened_joint_3: type fixed, parent z_401xr___encoder__401xr___encoder, child z_401xr___h2__l1___homelimit_switch__401xr___h2__l1___homelimit_switch, origin xyz=0 0 0 rpy=0 -0 0
- added joint z_group_2_fastened_joint_4: type fixed, parent z_401xr___carriage__401xr___carriage, child z_401xr___encoder_base_2__401xr___encoder_base_2_1, origin xyz=-0.0213302 -0.02125 -0.020468 rpy=0 -0 0
- added joint z_group_2_fastened_joint_5: type fixed, parent z_401xr___encoder_base_2__401xr___encoder_base_2_1, child z_401xr___encoder__401xr___encoder, origin xyz=0 0 0 rpy=0 -0 0
- added joint z_mounted_to_x_carriage: type fixed, parent 401xr___carriage__401xr___carriage, child z_c3_401xr__c3_401xr, origin xyz=-0.07188 0.13448 0.028645 rpy=-1.5708 0 0
- added joint z_slide: type prismatic, parent z_401xr_150_base__401xr_150_base, child z_401xr___carriage__401xr___carriage, origin xyz=0.09263 -0.04329 0.03002 rpy=3.141593 -1.570793 0, axis 1 0 0, limit lower=-0.05397 upper=0.09603 effort=1 velocity=1

Commit message: Make the Z stage a fixed column at the assembly centre
Re-root the 401XR 150 from the X carriage to root so it no longer rides
the XY slides: the column stays put at the assembly centre (footprint
centred on the X carriage mid position) and only z_slide moves its
carriage along world +Z.  Because the XY stages now sweep beneath the
fixed column, its base end was raised 2.5 mm so it floats ~2.1 mm above
the tallest swept feature (the X-base rails), which the collision sweep
verifies across all 125 configs.  The Z links leave the Y/X moving
groups, the kinematic-tree SVG draws the Z branch off root, the
collision SVG drops the Z sweep envelope, and the README/package.xml
describe the fixed column.

🤖 Generated with Codebuff
Co-Authored-By: Codebuff <noreply@codebuff.com>

File: urdf/parkerstage.urdf (robot description, URDF)
Before this commit: robot parkerstage, 36 links, 35 joints
Joints:
- removed joint z_mounted_to_x_carriage
- added joint z_mounted_to_root: type fixed, parent root, child z_c3_401xr__c3_401xr, origin xyz=-0.041268 -0.035307 0.168675 rpy=0 0 0

Commit message: Center the Z column in line with the XY assembly and guard its position
The fixed 401XR150 column was mounted 57.3 mm off the shared centre line of
the Y and X assemblies: the Z mount's footprint-centering term set the wrong
sign, leaving the column 57 mm south of the carriage centre in y (x was
already aligned).  Flip that term so the base footprint centre lands exactly
on the X carriage centre at q=0 -- the centre line shared by the plate, X
base and X carriage -- with the 125-config collision sweep still zero-overlap.

Add a Z CENTERED verify() guard that recomputes the footprint centre from the
meshes and asserts it coincides with the X carriage centre (the stroke,
mid-stroke and home guards are invariant to a planar mount shift, so this
closes that gap), alongside the Z INDEPENDENCE guard asserting no Z link
moves with the y/x slides.  Regenerate the URDF (z_mounted_to_root origin y
-0.035307 -> +0.021983) and the collision-geometry diagram.

🤖 Generated with Codebuff
Co-Authored-By: Codebuff <noreply@codebuff.com>

File: urdf/parkerstage.urdf (robot description, URDF)
Before this commit: robot parkerstage, 36 links, 35 joints
Joints:
- joint z_mounted_to_root: origin xyz=-0.041268 -0.035307 0.168675 rpy=0 0 0 -> xyz=-0.041267 0.021983 0.168675 rpy=0 0 0

Commit message: Re-center the fixed Z column on the XY mid-travel point and raise it 50 mm
Anchor the column's footprint on the centre of the XY travel envelope
(both slides at MID_STROKE) so it stays on the assembly centre line
across the full stroke instead of over the q=0 export datum, and lift
the whole Z assembly 50 mm in +z while preserving the ~2.1 mm designed
clearance over the swept X-base rails. Retarget the Z CENTERED guard to
the X carriage at mid-stroke.

Generated with Codebuff 🤖
Co-Authored-By: Codebuff <noreply@codebuff.com>

File: urdf/parkerstage.urdf (robot description, URDF)
Before this commit: robot parkerstage, 36 links, 35 joints
Joints:
- joint z_mounted_to_root: origin xyz=-0.041267 0.021983 0.168675 rpy=0 0 0 -> xyz=-0.020534 0.042715 0.218675 rpy=0 0 0
