Commit message: Rebuild XY stage from the corrected xyslideassy slide
Single-source both the Y and X axes from the corrected 200 mm slide
(xyslideassy): each stage clones the slide verbatim — the slider origin,
axis and [+48.370, +248.370] mm limits bracketed by the H3 limit switches,
with the seal bolted to each base and home at mid-stroke.  The Z column is
centred on the XY mid-travel point (X carriage body centre at mid-stroke),
raised clear of the tallest XY material, and guarded against drift, and all
mesh references are rewritten to local meshes.  verify() re-checks stroke,
limits-vs-slide, home, Z independence, slide direction, Z centring and a
125-config collision sweep (all pass).

🤖 Generated with Codebuff
Co-Authored-By: Codebuff <noreply@codebuff.com>

File: urdf/parkerstage.urdf (robot description, URDF)
Before this commit: robot parkerstage, 36 links, 35 joints
Links:
- removed link 401200xr__1_
- removed link 401200xr__3_
- removed link 401xr___carriage__401xr___carriage
- removed link 401xr___carriage__401xr___carriage_1
- removed link 401xr___carriage_end_caps__401xr___carriage_end_caps_1
- removed link 401xr___carriage_end_caps__401xr___carriage_end_caps_1_1
- removed link 401xr___carriage_end_caps__401xr___carriage_end_caps_2
- removed link 401xr___encoder__401xr___encoder
- removed link 401xr___encoder__401xr___encoder_1
- removed link 401xr___encoder_base_2__401xr___encoder_base_2
- removed link 401xr___encoder_base_2__401xr___encoder_base_2_1
- removed link 401xr___h2__l1___homelimit_switch__401xr___h2__l1___homelimit_switch
- removed link 401xr___h2__l1___homelimit_switch__401xr___h2__l1___homelimit_switch_1
- removed link 401xr___switch_flag__401xr___switch_flag
- removed link 401xr___switch_flag__401xr___switch_flag_1
- removed link plate
- removed link root
- added link x_401xr_200_seal_seal__401xr_200_seal_seal, mass 0.0224235; collision box size=0.3308 0.000644 0.019814; visual mesh filename=meshes/_401XR_200_Seal_seal__401XR_200_Seal_seal.stl scale=1 1 1
- added link x_401xr___carriage__401xr___carriage, mass 0.0634284; collision box size=0.0468 0.01725 0.039736; visual mesh filename=meshes/_401XR___Carriage__401XR___Carriage.stl scale=1 1 1
- added link x_401xr___carriage_end_caps__401xr___carriage_end_caps_1, mass 0.032373; collision box size=0.0941 0.0073 0.0338; visual mesh filename=meshes/_401XR___Carriage_End_Caps__401XR___Carriage_End_Cap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 scale=1 1 1
- added link x_401xr___carriage_end_caps__401xr___carriage_end_caps__1_, mass 1e-09
- added link x_401xr___encoder__401xr___encoder, mass 0.0346248; collision box size=0.0448 0.03188 0.0172; visual mesh filename=meshes/_401XR___Encoder__401XR___Encoder.stl scale=1 1 1
- added link x_401xr___encoder_base_2__401xr___encoder_base_2, mass 0.0031617; collision box size=0.0138 0.00735 0.0098; visual mesh filename=meshes/_401XR___Encoder_Base_2__401XR___Encoder_Base_2.stl scale=1 1 1
- added link x_401xr___h2__l1___homelimit_switch__401xr___h2__l1___homelimit_switch, mass 0.0047223; collision box size=0.034225 0.0088 0.0075; visual mesh filename=meshes/_401XR___H2__L1___Homelimit_Switch__401XR___H2__L1__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 scale=1 1 1
- added link x_401xr___switch_flag__401xr___switch_flag, mass 0.0009018; collision box size=0.01429 0.018034 0.006824; visual mesh filename=meshes/_401XR___Switch_Flag__401XR___Switch_Flag.stl scale=1 1 1
- added link x_root, mass 0.1463589; collision box size=0.056 0.3871 0.056; visual mesh filename=meshes/C3_401XR__C3_401XR.stl scale=1 1 1
- added link y_401xr_200_seal_seal__401xr_200_seal_seal, mass 0.0224235; collision box size=0.3308 0.000644 0.019814; visual mesh filename=meshes/_401XR_200_Seal_seal__401XR_200_Seal_seal.stl scale=1 1 1
- added link y_401xr___carriage__401xr___carriage, mass 0.0634284; collision box size=0.0468 0.01725 0.039736; visual mesh filename=meshes/_401XR___Carriage__401XR___Carriage.stl scale=1 1 1
- added link y_401xr___carriage_end_caps__401xr___carriage_end_caps_1, mass 0.032373; collision box size=0.0941 0.0073 0.0338; visual mesh filename=meshes/_401XR___Carriage_End_Caps__401XR___Carriage_End_Cap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 scale=1 1 1
- added link y_401xr___carriage_end_caps__401xr___carriage_end_caps__1_, mass 1e-09
- added link y_401xr___encoder__401xr___encoder, mass 0.0346248; collision box size=0.0448 0.03188 0.0172; visual mesh filename=meshes/_401XR___Encoder__401XR___Encoder.stl scale=1 1 1
- added link y_401xr___encoder_base_2__401xr___encoder_base_2, mass 0.0031617; collision box size=0.0138 0.00735 0.0098; visual mesh filename=meshes/_401XR___Encoder_Base_2__401XR___Encoder_Base_2.stl scale=1 1 1
- added link y_401xr___h2__l1___homelimit_switch__401xr___h2__l1___homelimit_switch, mass 0.0047223; collision box size=0.034225 0.0088 0.0075; visual mesh filename=meshes/_401XR___H2__L1___Homelimit_Switch__401XR___H2__L1__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 scale=1 1 1
- added link y_401xr___switch_flag__401xr___switch_flag, mass 0.0009018; collision box size=0.01429 0.018034 0.006824; visual mesh filename=meshes/_401XR___Switch_Flag__401XR___Switch_Flag.stl scale=1 1 1
- added link y_root, mass 0.1463589; collision box size=0.056 0.3871 0.056; visual mesh filename=meshes/C3_401XR__C3_401XR.stl scale=1 1 1
- link z_10851610__10851610: geometry collision box size=0.0397 0.034715 0.0188; visual mesh filename=package://parkerstage/meshes/z__10851610__10851610.stl scale=1 1 1
- link z_401xr_150_base__401xr_150_base: geometry collision box size=0.0397 0.03209 0.2658; visual mesh filename=package://parkerstage/meshes/z__401XR_150_Base__401XR_150_B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 scale=1 1 1
- link z_401xr_150_seal_seal__401xr_150_seal_seal: geometry collision box size=0.019814 0.000644 0.2808; visual mesh filename=package://parkerstage/meshes/z__401XR_150_Seal_seal__401XR_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 scale=1 1 1
- link z_401xr___150___d9___drive_screw__401xr___150___d9___drive_screw: geometry collision box size=0.0108 0.0108 0.2848; visual mesh filename=package://parkerstage/meshes/z__401XR___150___D9___Drive_Sc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 scale=1 1 1
- link z_401xr___carriage__401xr___carriage: geometry collision box size=0.0468 0.01725 0.039736; visual mesh filename=package://parkerstage/meshes/z__401XR___Carriage__401XR___C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 scale=1 1 1
- link z_401xr___carriage_end_caps__401xr___carriage_end_caps: geometry collision box size=0.0941 0.0073 0.0338; visual mesh filename=package://parkerstage/meshes/z__401XR___Carriage_End_Caps__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 scale=1 1 1
- link z_401xr___encoder__401xr___encoder: geometry collision box size=0.0448 0.03188 0.0172; visual mesh filename=package://parkerstage/meshes/z__401XR___Encoder__401XR___En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 scale=1 1 1
- link z_401xr___encoder_base_2__401xr___encoder_base_2: geometry collision box size=0.0098 0.00735 0.0138; visual mesh filename=package://parkerstage/meshes/z__401XR___Encoder_Base_2__401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 scale=1 1 1
- link z_401xr___encoder_base_2__401xr___encoder_base_2_1: geometry collision box size=0.0138 0.00735 0.0098; visual mesh filename=package://parkerstage/meshes/z__401XR___Encoder_Base_2__401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 scale=1 1 1
- link z_401xr___h2__l1___homelimit_switch__401xr___h2__l1___homelimit_switch: geometry collision box size=0.034225 0.0088 0.0075; visual mesh filename=package://parkerstage/meshes/z__401XR___H2__L1___Homelimit_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 scale=1 1 1
- link z_401xr___h2__l2___homelimit_switch__401xr___h2__l2___homelimit_switch_1: geometry collision box size=0.0075 0.0088 0.205225; visual mesh filename=package://parkerstage/meshes/z__401XR___H2__L2___Homelimit_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 scale=1 1 1
- link z_401xr___switch_flag__401xr___switch_flag: geometry collision box size=0.01429 0.018034 0.006824; visual mesh filename=package://parkerstage/meshes/z__401XR___Switch_Flag__401XR_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 scale=1 1 1
- link z_401xr_back_ballscrew_holder__401xr_back_ballscrew_holder: geometry collision box size=0.0318 0.0228 0.0078; visual mesh filename=package://parkerstage/meshes/z__401XR_Back_Ballscrew_Holder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 scale=1 1 1
- link z_401xr_coupling_housing__401xr_coupling_housing: geometry collision box size=0.0397 0.041675 0.0488; visual mesh filename=package://parkerstage/meshes/z__401XR_Coupling_Housing__401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 scale=1 1 1
- link z_401xr_front_ballscrew_holder__401xr_front_ballscrew_holder: geometry collision box size=0.0318 0.0228 0.0188; visual mesh filename=package://parkerstage/meshes/z__401XR_Front_Ballscrew_Holde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 scale=1 1 1
- link z_c3_401xr__c3_401xr: geometry collision box size=0.0178 0.017772 0.0248; visual mesh filename=package://parkerstage/meshes/z_C3_401XR__C3_401XR.stl scale=1 1 1
- link z_m2___sm_16__m2___sm_16: geometry collision box size=0.02875 0.028706 0.0017; visual mesh filename=package://parkerstage/meshes/z_M2___SM_16__M2___SM_16.stl scale=1 1 1
Joints:
- removed joint base1_fixed_to_root
- removed joint base2_mounted_to_plate
- removed joint carriage2_fastened_joint
- removed joint carriage2_fastened_joint_1
- removed joint carriage2_fastened_joint_2
- removed joint carriage2_fastened_joint_3
- removed joint carriage2_fastened_joint_4
- removed joint carriage_fastened_joint
- removed joint carriage_fastened_joint_1
- removed joint carriage_fastened_joint_2
- removed joint carriage_fastened_joint_3
- removed joint carriage_fastened_joint_4
- removed joint carriage_fastened_joint_5
- removed joint fastened_1
- added joint x_carriage_fastened_joint: type fixed, parent x_401xr___carriage__401xr___carriage, child x_401xr___encoder__401xr___encoder, origin xyz=0 0 0 rpy=-8.27902e-64 6.71674e-32 -2.46519e-32
- added joint x_carriage_fastened_joint_1: type fixed, parent x_401xr___switch_flag__401xr___switch_flag, child x_401xr___encoder_base_2__401xr___encoder_base_2, origin xyz=0 0 0 rpy=-8.27902e-64 6.71674e-32 -2.46519e-32
- added joint x_carriage_fastened_joint_2: type fixed, parent x_401xr___switch_flag__401xr___switch_flag, child x_401xr___carriage_end_caps__401xr___carriage_end_caps__1_, origin xyz=0 0 0 rpy=-8.27902e-64 6.71674e-32 -2.46519e-32
- added joint x_carriage_fastened_joint_3: type fixed, parent x_401xr___carriage_end_caps__401xr___carriage_end_caps__1_, child x_401xr___carriage_end_caps__401xr___carriage_end_caps_1, origin xyz=0 0 0 rpy=-8.27902e-64 6.71674e-32 -2.46519e-32
- added joint x_carriage_fastened_joint_4: type fixed, parent x_401xr___carriage_end_caps__401xr___carriage_end_caps_1, child x_401xr___carriage__401xr___carriage, origin xyz=0 0 0 rpy=-8.27902e-64 6.71674e-32 -2.46519e-32
- added joint x_carriage_fastened_joint_5: type fixed, parent x_401xr___encoder__401xr___encoder, child x_401xr___h2__l1___homelimit_switch__401xr___h2__l1___homelimit_switch, origin xyz=0 0 0 rpy=-8.27902e-64 6.71674e-32 -2.46519e-32
- added joint x_onto_ycarriage: type fixed, parent y_401xr___switch_flag__401xr___switch_flag, child x_root, origin xyz=-0.094994 -0.01562 0.07966 rpy=-1.5708 0 0
- added joint x_seal_to_base: type fixed, parent x_root, child x_401xr_200_seal_seal__401xr_200_seal_seal, origin xyz=0.061544 0.052688 -0.01562 rpy=1.5708 0 -1.5708
- added joint y_carriage_fastened_joint: type fixed, parent y_401xr___carriage__401xr___carriage, child y_401xr___encoder__401xr___encoder, origin xyz=0 0 0 rpy=-8.27902e-64 6.71674e-32 -2.46519e-32
- added joint y_carriage_fastened_joint_1: type fixed, parent y_401xr___switch_flag__401xr___switch_flag, child y_401xr___encoder_base_2__401xr___encoder_base_2, origin xyz=0 0 0 rpy=-8.27902e-64 6.71674e-32 -2.46519e-32
- added joint y_carriage_fastened_joint_2: type fixed, parent y_401xr___switch_flag__401xr___switch_flag, child y_401xr___carriage_end_caps__401xr___carriage_end_caps__1_, origin xyz=0 0 0 rpy=-8.27902e-64 6.71674e-32 -2.46519e-32
- added joint y_carriage_fastened_joint_3: type fixed, parent y_401xr___carriage_end_caps__401xr___carriage_end_caps__1_, child y_401xr___carriage_end_caps__401xr___carriage_end_caps_1, origin xyz=0 0 0 rpy=-8.27902e-64 6.71674e-32 -2.46519e-32
- added joint y_carriage_fastened_joint_4: type fixed, parent y_401xr___carriage_end_caps__401xr___carriage_end_caps_1, child y_401xr___carriage__401xr___carriage, origin xyz=0 0 0 rpy=-8.27902e-64 6.71674e-32 -2.46519e-32
- added joint y_carriage_fastened_joint_5: type fixed, parent y_401xr___encoder__401xr___encoder, child y_401xr___h2__l1___homelimit_switch__401xr___h2__l1___homelimit_switch, origin xyz=0 0 0 rpy=-8.27902e-64 6.71674e-32 -2.46519e-32
- added joint y_seal_to_base: type fixed, parent y_root, child y_401xr_200_seal_seal__401xr_200_seal_seal, origin xyz=0.061544 0.052688 -0.01562 rpy=1.5708 0 -1.5708
- added joint y_to_root: type fixed, parent root, child y_root
- joint x_slide: axis 1 0 0 -> -1 0 0; child 401xr___encoder__401xr___encoder -> x_401xr___switch_flag__401xr___switch_flag; limit lower=-0.079267 upper=0.120733 effort=1 velocity=1 -> lower=0.04837 upper=0.24837 effort=1 velocity=1; origin xyz=0 -0.03405 -0.02135 rpy=1.5708 0 1.570796 -> xyz=0.094994 0.031338 -0.01562 rpy=1.5708 0 -1.5708; parent 401200xr__3_ -> x_root
- joint y_slide: axis 0 1 0 -> -1 0 0; child plate -> y_401xr___switch_flag__401xr___switch_flag; limit lower=-0.079267 upper=0.120733 effort=1 velocity=1 -> lower=0.04837 upper=0.24837 effort=1 velocity=1; origin xyz=0 -0.03375 0.018771 rpy=0 0 0 -> xyz=0.094994 0.031338 -0.01562 rpy=1.5708 0 -1.5708; parent 401200xr__1_ -> y_root
- joint z_mounted_to_root: origin xyz=-0.020534 0.042715 0.218675 rpy=0 0 0 -> xyz=-0.019104 0.161395 0.329316 rpy=0 0 0
- joint z_slide: limit lower=-0.05397 upper=0.09603 effort=1 velocity=1 -> lower=-0.11658 upper=0.03342 effort=1 velocity=1
